File: hardware/designs/light2-harness-r02/schematic.kicad_sch (KiCad schematic)
At the start: 45 parts, among them J2 Olimex P4 EXT1, J3 Olimex P4 EXT2, U1 SN74LVC244AN, U2 SN74LVC244AN, U3 SN74LV125AN, U4 SN74LV125AN

Commit message: HW-001: promote canonical physical harness schematic
Parts:
- U1, U2: symbol HW001_Draft:SN74LVC244AN -> Physical_DIP:SN74LVC244AN_DIP_TOP
- U3, U4: symbol HW001_Draft:SN74LV125AN -> Physical_DIP:SN74LV125AN_DIP_TOP
Connections:
- net agon-3v3: now also C1.2, C2.2, C3.2, R26.2; no longer C1.1, C2.1, C3.1, R26.1
- net ground: now also C1.1, C2.1, C3.1, C4.1; no longer C1.2, C2.2, C3.2, C4.2
- net p4-3v3: now also C4.2; no longer C4.1
- net at R13.1: now also JO1.7 (Pin_7), R24.2; no longer U4.11 (4Y)
- net at U1.19 (2OE_N), U2.1 (1OE_N), U4.6 (2Y): now also R26.1; no longer R26.2
- new net: R13.2, U4.11 (4Y)
- no-connect marks 50 -> 0
Other:
- note added: "R1 220"
- note added: "R10 220"
- note added: "R11 220"
- note added: "R12 220"
- note added: "R13 220"
- note added: "R14 47k"
- note added: "R15 47k"
- note added: "R16 47k"
- note added: "R17 47k"
- note added: "R18 47k"
- note added: "R19 47k"
- note added: "R2 220"
- note added: "R20 47k"
- note added: "R21 47k"
- note added: "R22 10k"
- note added: "R23 10k"
- note added: "R24 10k"
- note added: "R25 10k"
- note added: "R26 10k"
- note added: "R27 10k"
- note added: "R28 10k"
- note added: "R29 10k"
- note added: "R3 220"
- note added: "R30 10k"
- note added: "R31 10k"
- note added: "R4 220"
- note added: "R5 220"
- note added: "R6 220"
- note added: "R7 220"
- note added: "R8 220"
- note added: "R9 220"
- title: Light 2 harness r02 — human electrical schematic -> Light 2 harness r02 — PHYSICAL TOP-VIEW DIP DIRECT-WIRE AID
- moved on the sheet: C1, C2, C3, C4, C5, C6, J2, J3, JE1, JO1
