File: hardware/designs/light2-harness-r02/signal-views/generated/02_schematic_startup-and-fail-safe-bias-network.kicad_sch (KiCad schematic)
At the start: 45 parts, among them J2 ESP32-P4 Right Header (EXT1), J3 ESP32-P4 Left Header (EXT2), U1 SN74LVC244AN, U2 SN74LVC244AN, U3 SN74LV125AN, U4 SN74LV125AN

Commit message: HW-001: freeze r02 schematic and ordered signal views
Connections:
- net at R11.1: no longer U3.3 (1Y)
- net at R5.1: no longer U2.18 (1Y1)
- net at R13.2: no longer U4.11 (4Y)
- net at R6.1: no longer U2.16 (1Y2)
- net at R7.1: no longer U2.14 (1Y3)
- net at U2.12 (1Y4): no longer R8.1
- net at U2.2 (1A1): no longer JO1.11 (Pin_11)
- net at U2.4 (1A2): no longer JE1.11 (Pin_11)
- net at U2.6 (1A3): no longer JO1.12 (Pin_12)
- net at U2.8 (1A4): no longer JE1.12 (Pin_12)
- net at R3.1: no longer U1.16 (1Y2)
- net at R1.1: no longer U1.18 (1Y1)
- net at R2.1: no longer U1.3 (2Y4)
- net at R10.1: no longer U1.9 (2Y1)
- net at R12.1: no longer U3.6 (2Y)
- net at R4.1: no longer U1.5 (2Y3)
- net at R9.1: no longer U1.7 (2Y2)
- net at JO1.10 (Pin_10): no longer U1.4 (1A2)
- net at JO1.9 (Pin_9): no longer U1.2 (1A1)
- net at JE1.7 (Pin_7): no longer U1.13 (2A2)
- net at JE1.8 (Pin_8): no longer U1.11 (2A1)
- now unconnected: JE1.10 (Pin_10), JE1.9 (Pin_9), R11.2, R12.2, U1.15 (2A3), U1.17 (2A4)
- no-connect marks 50 -> 0
Other:
- title: Light 2 harness r02 — PHYSICAL TOP-VIEW DIP DIRECT-WIRE AID -> Light 2 harness r02 — Startup and fail-safe bias network — FUNCTION VIEW, NOT AUTHORITY
